Commit message: update 9_30

File: robot_description/urdf/robot.urdf (robot description, URDF)
Before this commit: robot my_robot, 7 links, 6 joints
Links:
- added link aruco_marker_frame; visual box size=0.18 0.18 0.03
Joints:
- added joint aruco_marker_joint: type fixed, parent aruco_marker_frame, child base_link, origin xyz=0.0 0 -0.13 rpy=0 0 0
- joint camera_joint: child base_link -> camera_link; origin xyz=-0.27 0 -0.09 rpy=0 0 0 -> xyz=0.27 0 0.09 rpy=0 0 0; parent camera_link -> base_link
